File: FreeBoard.kicad_pcb (KiCad board)
At the start: 2 copper layers, 313 x 150 mm, 128 parts, among them SW1 SW_Push, SW10 SW_Push, SW11 SW_Push, SW12 SW_Push, SW13 SW_Push, SW14 SW_Push, SW15 SW_Push, SW16 SW_Push, SW17 SW_Push, SW18 SW_Push, SW19 SW_Push, SW2 SW_Push, SW20 SW_Push, SW21 SW_Push, SW22 SW_Push, SW23 SW_Push, SW24 SW_Push, SW25 SW_Push, SW26 SW_Push, SW27 SW_Push, SW28 SW_Push, SW29 SW_Push, SW3 SW_Push, SW30 SW_Push, SW31 SW_Push, SW32 SW_Push, SW33 SW_Push, SW34 SW_Push, SW35 SW_Push, SW36 SW_Push, SW37 SW_Push, SW38 SW_Push, SW39 SW_Push, SW4 SW_Push, SW40 SW_Push, SW41 SW_Push, SW42 SW_Push, SW43 SW_Push, SW44 SW_Push, SW45 SW_Push, SW46 SW_Push, SW47 SW_Push, SW48 SW_Push, SW49 SW_Push, SW5 SW_Push, SW50 SW_Push, SW51 SW_Push, SW52 SW_Push, SW53 SW_Push, SW54 SW_Push, SW55 SW_Push, SW56 SW_Push, SW57 SW_Push, SW58 SW_Push, SW59 SW_Push, SW6 SW_Push, SW60 SW_Push, SW61 SW_Push, SW62 SW_Push, SW63 RotaryEncoder_Switch, SW64 RotaryEncoder_Switch, SW65 RotaryEncoder_Switch, SW7 SW_Push, SW8 SW_Push, SW9 SW_Push, U2 Pico

Commit message: Add files via upload
Connections:
- SW63 pad C: Net-(SW63-PadC) -> GND
- SW63 pad S2: Net-(SW63-PadC) -> GND
- SW64 pad C: Net-(SW63-PadC) -> GND
- SW64 pad S2: Net-(SW63-PadC) -> GND
- SW65 pad C: Net-(SW63-PadC) -> GND
- SW65 pad S2: Net-(SW63-PadC) -> GND
- U2 pad 13: unconnected-(U2-GND-Pad13) -> GND
- U2 pad 18: unconnected-(U2-GND-Pad18)_1 -> GND
- U2 pad 23: unconnected-(U2-GND-Pad23)_1 -> GND
- U2 pad 28: Net-(SW63-PadC) -> GND
- U2 pad 3: unconnected-(U2-GND-Pad3)_1 -> GND
- U2 pad 38: unconnected-(U2-GND-Pad38)_1 -> GND
- U2 pad 42: unconnected-(U2-GND-Pad42) -> GND
- U2 pad 8: unconnected-(U2-GND-Pad8)_1 -> GND
Routing:
- net GND: track 0.00 -> 358.7 mm, vias 0 -> 4
- net Net-(SW63-PadC): track 271.1 -> 0.00 mm
